Commit message: feat(graspable): add basic object transfer (move_object_to_pose)

File: src/python/arcor2_ur/data/urdf/ur5e.urdf (robot description, URDF)
Before this commit: robot ur5e, 13 links, 12 joints
Links:
- added link onrobot_vgc10_base_link; collision mesh filename=file:///mnt/c/Users/Office/Desktop/diplomka/kod/arcor2-ur5e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; visual mesh filename=file:///mnt/c/Users/Office/Desktop/diplomka/kod/arcor2-ur5e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
- added link suction; collision mesh filename=file:///mnt/c/Users/Office/Desktop/diplomka/kod/arcor2-ur5e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; visual mesh filename=file:///mnt/c/Users/Office/Desktop/diplomka/kod/arcor2-ur5e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
- link base_link_inertia: geometry collision mesh filename=file:///mnt/c/Users/Office/Desktop/diplomka/kod/arcor2-ur5e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; visual mesh filename=file:///mnt/c/Users/Office/Desktop/diplomka/kod/arcor2-ur5e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
- link forearm_link: geometry collision mesh filename=file:///mnt/c/Users/Office/Desktop/diplomka/kod/arcor2-ur5e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; visual mesh filename=file:///mnt/c/Users/Office/Desktop/diplomka/kod/arcor2-ur5e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
- link shoulder_link: geometry collision mesh filename=file:///mnt/c/Users/Office/Desktop/diplomka/kod/arcor2-ur5e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; visual mesh filename=file:///mnt/c/Users/Office/Desktop/diplomka/kod/arcor2-ur5e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
- link upper_arm_link: geometry collision mesh filename=file:///mnt/c/Users/Office/Desktop/diplomka/kod/arcor2-ur5e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; visual mesh filename=file:///mnt/c/Users/Office/Desktop/diplomka/kod/arcor2-ur5e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
- link wrist_1_link: geometry collision mesh filename=file:///mnt/c/Users/Office/Desktop/diplomka/kod/arcor2-ur5e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; visual mesh filename=file:///mnt/c/Users/Office/Desktop/diplomka/kod/arcor2-ur5e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
- link wrist_2_link: geometry collision mesh filename=file:///mnt/c/Users/Office/Desktop/diplomka/kod/arcor2-ur5e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; visual mesh filename=file:///mnt/c/Users/Office/Desktop/diplomka/kod/arcor2-ur5e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
- link wrist_3_link: geometry collision mesh filename=file:///mnt/c/Users/Office/Desktop/diplomka/kod/arcor2-ur5e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; visual mesh filename=file:///mnt/c/Users/Office/Desktop/diplomka/kod/arcor2-ur5e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
Joints:
- added joint vgc10_suction_joint: type fixed, parent onrobot_vgc10_base_link, child suction, origin xyz=0 0 0.094901 rpy=0 0 0
- added joint wrist_3_to_vgc10_joint: type fixed, parent wrist_3_link, child onrobot_vgc10_base_link, origin xyz=0 0 0 rpy=0 0 0
- joint wrist_3-flange: parent wrist_3_link -> tool0
- joint wrist_3_link-ft_frame: parent wrist_3_link -> tool0

Commit message: feat: add graspable first attach and detach algorithm, added stl base a suction cup

File: src/python/arcor2_ur/data/urdf/ur5e.urdf (robot description, URDF)
Before this commit: robot ur5e, 15 links, 14 joints
Links:
- removed link onrobot_vgc10_base_link
- removed link suction
- link base_link_inertia: geometry collision mesh filename=package://meshes/ur5e/collision/base.stl; visual mesh filename=package://meshes/ur5e/visual/base.dae
- link forearm_link: geometry collision mesh filename=package://meshes/ur5e/collision/forearm.stl; visual mesh filename=package://meshes/ur5e/visual/forearm.dae
- link shoulder_link: geometry collision mesh filename=package://meshes/ur5e/collision/shoulder.stl; visual mesh filename=package://meshes/ur5e/visual/shoulder.dae
- link upper_arm_link: geometry collision mesh filename=package://meshes/ur5e/collision/upperarm.stl; visual mesh filename=package://meshes/ur5e/visual/upperarm.dae
- link wrist_1_link: geometry collision mesh filename=package://meshes/ur5e/collision/wrist1.stl; visual mesh filename=package://meshes/ur5e/visual/wrist1.dae
- link wrist_2_link: geometry collision mesh filename=package://meshes/ur5e/collision/wrist2.stl; visual mesh filename=package://meshes/ur5e/visual/wrist2.dae
- link wrist_3_link: geometry collision mesh filename=package://meshes/ur5e/collision/wrist3.stl; visual mesh filename=package://meshes/ur5e/visual/wrist3.dae
Joints:
- removed joint vgc10_suction_joint
- removed joint wrist_3_to_vgc10_joint
- joint wrist_3-flange: parent tool0 -> wrist_3_link
- joint wrist_3_link-ft_frame: parent tool0 -> wrist_3_link
